Commit message: Update dynamixel_head_hardware.xacro

File: hexapod_description/urdf/dynamixel_head_hardware.xacro (robot description, xacro)
@@ -33,5 +33,5 @@
         <origin xyz="0 0 0 " rpy="0 0 0" />
         <geometry>
-          <mesh filename="package://rbx2_description/meshes/F10.stl" scale="${DYNAMIXEL_MESH_SCALE} ${DYNAMIXEL_MESH_SCALE} ${DYNAMIXEL_MESH_SCALE}"/>
+          <mesh filename="package://hexapod_description/meshes/phantomX/F10.stl" scale="${DYNAMIXEL_MESH_SCALE} ${DYNAMIXEL_MESH_SCALE} ${DYNAMIXEL_MESH_SCALE}"/>
         </geometry>
         <material name="${color}"/>

Commit message: Update dynamixel_head_hardware.xacro

File: hexapod_description/urdf/dynamixel_head_hardware.xacro (robot description, xacro)
@@ -62,5 +62,5 @@
         <origin xyz="0 0 0 " rpy="0 0 0" />
         <geometry>
-          <mesh filename="package://rbx2_description/meshes/F3.stl" scale="${DYNAMIXEL_MESH_SCALE} ${DYNAMIXEL_MESH_SCALE} ${DYNAMIXEL_MESH_SCALE}"/>
+          <mesh filename="package://hexapod_description/meshes/phantomX/F3.stl" scale="${DYNAMIXEL_MESH_SCALE} ${DYNAMIXEL_MESH_SCALE} ${DYNAMIXEL_MESH_SCALE}"/>
         </geometry>
         <material name="${color}"/>
@@ -91,5 +91,5 @@
         <origin xyz="0 0 0 " rpy="0 0 0" />
         <geometry>
-          <mesh filename="package://rbx2_description/meshes/ax12.stl" scale="${DYNAMIXEL_MESH_SCALE} ${DYNAMIXEL_MESH_SCALE} ${DYNAMIXEL_MESH_SCALE}"/>
+          <mesh filename="package://hexapod_description/meshes/phantomX/ax12.stl" scale="${DYNAMIXEL_MESH_SCALE} ${DYNAMIXEL_MESH_SCALE} ${DYNAMIXEL_MESH_SCALE}"/>
         </geometry>
         <material name="Black"/>
@@ -122,5 +122,5 @@
         <origin xyz="0 0 0 " rpy="0 0 0" />
         <geometry>
-          <mesh filename="package://rbx2_description/meshes/F3.stl" scale="${DYNAMIXEL_MESH_SCALE} ${DYNAMIXEL_MESH_SCALE} ${DYNAMIXEL_MESH_SCALE}"/>
+          <mesh filename="package://hexapod_description/meshes/phantomX/F3.stl" scale="${DYNAMIXEL_MESH_SCALE} ${DYNAMIXEL_MESH_SCALE} ${DYNAMIXEL_MESH_SCALE}"/>
         </geometry>
         <material name="${color}"/>
@@ -153,5 +153,5 @@
         <origin xyz="0 0 0 " rpy="0 0 0" />
         <geometry>
-          <mesh filename="package://rbx2_description/meshes/F4.stl" scale="${DYNAMIXEL_MESH_SCALE} ${DYNAMIXEL_MESH_SCALE} ${DYNAMIXEL_MESH_SCALE}"/>
+          <mesh filename="package://hexapod_description/meshes/phantomX/F4.stl" scale="${DYNAMIXEL_MESH_SCALE} ${DYNAMIXEL_MESH_SCALE} ${DYNAMIXEL_MESH_SCALE}"/>
         </geometry>
         <material name="${color}"/>
@@ -184,5 +184,5 @@
         <origin xyz="0 0 0 " rpy="0 0 0" />
         <geometry>
-          <mesh filename="package://rbx2_description/meshes/F2.stl" scale="${DYNAMIXEL_MESH_SCALE} ${DYNAMIXEL_MESH_SCALE} ${DYNAMIXEL_MESH_SCALE}"/>
+          <mesh filename="package://hexapod_description/meshes/phantomX/F2.stl" scale="${DYNAMIXEL_MESH_SCALE} ${DYNAMIXEL_MESH_SCALE} ${DYNAMIXEL_MESH_SCALE}"/>
         </geometry>
         <material name="${color}"/>
