Commit message: Update phantomX_model.xacro

File: hexapod_description/urdf/phantomX_model.xacro (robot description, xacro)
@@ -8,4 +8,7 @@
 	<xacro:property name="femur_length" value="0.065" />
 	<xacro:property name="tibia_length" value="0.133" />
+	<xacro:property name="head_offset_x" value="0.0475" />
+        <xacro:property name="head_offset_y" value="0.0036" />
+        <xacro:property name="head_offset_z" value="0.875" />
     <gazebo>
         <plugin name="gazebo_ros_control" filename="libgazebo_ros_control.so">
@@ -50,4 +53,8 @@
         <material>Gazebo/DarkGrey</material>
     </gazebo>
+     <!-- Attach the pan and tilt head -->
+    <head name="head_base" parent="body_link" color="White">
+      <origin xyz="${head_offset_x} ${head_offset_y} ${head_offset_z}" rpy="0 0 ${PI}" />
+    </head>
 	<!-- Head Pan and Tilt properties -->
 	<joint name="head_pan_joint" type="revolute">

Commit message: Update phantomX_model.xacro

File: hexapod_description/urdf/phantomX_model.xacro (robot description, xacro)
@@ -8,7 +8,4 @@
 	<xacro:property name="femur_length" value="0.065" />
 	<xacro:property name="tibia_length" value="0.133" />
-	<xacro:property name="head_offset_x" value="0.0475" />
-        <xacro:property name="head_offset_y" value="0.0036" />
-        <xacro:property name="head_offset_z" value="0.875" />
     <gazebo>
         <plugin name="gazebo_ros_control" filename="libgazebo_ros_control.so">
@@ -53,105 +50,4 @@
         <material>Gazebo/DarkGrey</material>
     </gazebo>
-     <!-- Attach the pan and tilt head -->
-    <head name="head_base" parent="body_link" color="White">
-      <origin xyz="${head_offset_x} ${head_offset_y} ${head_offset_z}" rpy="0 0 ${PI}" />
-    </head>
-	<!-- Head Pan and Tilt properties -->
-	<joint name="head_pan_joint" type="revolute">
-		<parent link="body_link"/>
-		<child link="head_pan_link"/>
-		<axis xyz="0.0 0.0 1.0" />
-		<origin xyz="0.145 0.0 0.080" />
-		<limit lower="-${3.14}" upper="${3.14}" effort="10000" velocity="100" />
-	</joint>
-	<link name="head_pan_link">
-        <inertial>
-            <origin xyz="0.0 0.0 0.0" rpy="0.0 0.0 0.0" />
-            <mass value="0.00001"/>
-            <inertia
-                ixx="1.0" ixy="0.0"  ixz="0.0"
-                iyy="1.0" iyz="0.0"
-                izz="1.0" />
-        </inertial>
-    </link>
-	<joint name="head_tilt_joint" type="revolute">
-		<parent link="head_pan_link"/>
-		<child link="head_tilt_link"/>
-		<axis xyz="0.0 1.0 0.0" />
-		<origin xyz="0.0 0.0 0.020" />
-		<limit lower="-${3.14}" upper="${3.14}" effort="10000" velocity="100" />
-	</joint>
-	<link name="head_tilt_link">
-        <inertial>
-            <origin xyz="0.0 0.0 0.0" rpy="0.0 0.0 0.0" />
-            <mass value="0.00001"/>
-            <inertia
-                ixx="1.0" ixy="0.0"  ixz="0.0"
-                iyy="1.0" iyz="0.0"
-                izz="1.0" />
-        </inertial>
-    </link>
-	<!-- Camera properties -->
-	<joint name="camera_rgb_joint" type="fixed">
-		<parent link="head_tilt_link" />
-		<child link="camera_rgb_optical_frame" />
-		<origin xyz="0.0 0.0 0.0" rpy="${pi/2} ${pi} ${pi/2}" />
-	</joint>
-	<link name="camera_rgb_optical_frame">
-        <inertial>
-            <origin xyz="0.0 0.0 0.0" rpy="0.0 0.0 0.0" />
-            <mass value="0.00001"/>
-            <inertia
-                ixx="1.0" ixy="0.0"  ixz="0.0"
-                iyy="1.0" iyz="0.0"
-                izz="1.0" />
-        </inertial>
-    </link>
-	<joint name="camera_depth_joint" type="fixed">
-		<parent link="head_tilt_link" />
-		<child link="camera_depth_optical_frame" />
-		<origin xyz="0.0 0.0 0.0" rpy="${pi/2} ${pi} ${pi/2}" />
-	</joint>
-	<link name="camera_depth_optical_frame" >
-        <inertial>
-            <origin xyz="0.0 0.0 0.0" rpy="0.0 0.0 0.0" />
-            <mass value="0.00001"/>
-            <inertia
-                ixx="1.0" ixy="0.0"  ixz="0.0"
-                iyy="1.0" iyz="0.0"
-                izz="1.0" />
-        </inertial>
-    </link>
-<joint name="camera_depth_frame" type="fixed">
-	<parent link="head_tilt_link" />
-	<child link="camera_depth_frame_link" />
-	<origin xyz="0.0 0.0 0.0" />
-</joint>
-<link name="camera_depth_frame_link" >
-        <inertial>
-            <origin xyz="0.0 0.0 0.0" rpy="0.0 0.0 0.0" />
-            <mass value="0.00001"/>
-            <inertia
-                ixx="1.0" ixy="0.0"  ixz="0.0"
-                iyy="1.0" iyz="0.0"
-                izz="1.0" />
-        </inertial>
-    </link>
-	<!-- IMU properties
-	<joint name="imu_joint" type="fixed">
-		<parent link="base_link" />
-		<child link="imu_link" />
-		<origin xyz="0.0 0.0 0.0" rpy="0.0 0.0 0.0" />
-	</joint>
-	<link name="imu_link">
-        <inertial>
-            <origin xyz="0.0 0.0 0.0" rpy="0.0 0.0 0.0" />
-            <mass value="0.00001"/>
-            <inertia
-                ixx="1.0" ixy="0.0"  ixz="0.0"
-                iyy="1.0" iyz="0.0"
-                izz="1.0" />
-        </inertial>
-    </link>-->
 	<!-- Joint properties -->
 	<xacro:property name="joint_lower_limit" value="-${3.14}" />

Commit message: Update phantomX_model.xacro

File: hexapod_description/urdf/phantomX_model.xacro (robot description, xacro)
@@ -8,4 +8,7 @@
 	<xacro:property name="femur_length" value="0.065" />
 	<xacro:property name="tibia_length" value="0.133" />
+	<xacro:property name="head_offset_x" value="0.0475" />
+        <xacro:property name="head_offset_y" value="0.0036" />
+        <xacro:property name="head_offset_z" value="0.875" />
     <gazebo>
         <plugin name="gazebo_ros_control" filename="libgazebo_ros_control.so">
@@ -50,4 +53,8 @@
         <material>Gazebo/DarkGrey</material>
     </gazebo>
+ 	<!-- Attach the pan and tilt head -->
+   	<head name="head_base" parent="torso" color="White">
+      		<origin xyz="${head_offset_x} ${head_offset_y} ${head_offset_z}" rpy="0 0 ${PI}" />
+   	</head>
 	<!-- Joint properties -->
 	<xacro:property name="joint_lower_limit" value="-${3.14}" />

Commit message: Update phantomX_model.xacro

File: hexapod_description/urdf/phantomX_model.xacro (robot description, xacro)
@@ -51,4 +51,37 @@
         </inertial>
     </link>
+    <joint name="lidar_joint" type="fixed">
+        <parent link="body_link" />
+        <child link="lidar_link" />
+        <origin xyz="0.2 0.0 0.0" rpy="0.0 0.0 0.0" />
+    </joint>
+	<link name="lidar_link">
+			<visual>
+	  			<origin	xyz="0.0 0.0 0.0" rpy="0.0 0.0 0.0" />
+      			<geometry>
+        			<mesh filename="package://hexapod_description/meshes/phantomX/xv-11_lidar.stl" scale="0.001 0.001 0.001"/>
+      			</geometry>
+				<material name="">
+					<color rgba="0.7 0.7 0.7 1" />
+				</material>
+			</visual>
+			<collision>
+			<geometry>
+        			<mesh filename="package://hexapod_description/meshes/phantomX/xv-11_lidar.stl" scale="0.001 0.001 0.001"/>
+      			</geometry>
+            <origin xyz="0.0 0.0 0.0" rpy="0.0 0.0 0.0"/>
+            <material name="">
+                <color rgba="0.7 0.7 0.7 1"/>
+            </material>
+        </collision>
+        <inertial>
+            <origin xyz="0.0 0.0 0.0" rpy="0.0 0.0 0.0" />
+            <mass value="0.00001"/>
+            <inertia
+                ixx="1.0" ixy="0.0"  ixz="0.0"
+                iyy="1.0" iyz="0.0"
+                izz="1.0" />
+        </inertial>
+    </link>
     <gazebo reference="body_link">
         <material>Gazebo/DarkGrey</material>
