Commit message: modified:   hexapod_bringup/launch/components/rtabmap_AC.launch 	modified:   hexapod_description/params/phantomX.yaml 	modified:   hexapod_description/rviz_prefs/urdf.rviz 	modified:   hexapod_description/urdf/pan_tilt_head_xtion.urdf.xacro 	modified:   hexapod_description/urdf/phantomX_model.xacro

File: hexapod_description/urdf/pan_tilt_head_xtion.urdf.xacro (robot description, xacro)
@@ -5,6 +5,6 @@
   <property name="camera_offset_z" value="0.06" />
   <property name="camera_mesh_scale" value="1.0" />
-  <xacro:include filename="$(find hexapod_description)/urdf/pi_robot/dynamixel_head_hardware.xacro" />
-  <xacro:include filename="$(find hexapod_description)/urdf/pi_robot/xtion.urdf.xacro" />
+  <xacro:include filename="$(find hexapod_description)/urdf/dynamixel_head_hardware.xacro" />
+  <xacro:include filename="$(find hexapod_description)/urdf/xtion.urdf.xacro" />
   <macro name="head" params="parent name color *origin">
     <!-- head base joint -->

File: hexapod_description/urdf/phantomX_model.xacro (robot description, xacro)
@@ -8,7 +8,7 @@
 	<xacro:property name="femur_length" value="0.065" />
 	<xacro:property name="tibia_length" value="0.133" />
-	<xacro:property name="head_offset_x" value="0.0475" />
-        <xacro:property name="head_offset_y" value="0.0036" />
-        <xacro:property name="head_offset_z" value="0.875" />
+	<xacro:property name="head_offset_x" value="0.065" />
+  <xacro:property name="head_offset_y" value="0.000" />
+  <xacro:property name="head_offset_z" value="0.000" />
     <gazebo>
         <plugin name="gazebo_ros_control" filename="libgazebo_ros_control.so">
@@ -16,5 +16,5 @@
         </plugin>
     </gazebo>
-    <xacro:include filename="$(find rbx2_description)/urdf/pi_robot/pan_tilt_head_xtion.urdf.xacro" />
+    <xacro:include filename="$(find hexapod_description)/urdf/pan_tilt_head_xtion.urdf.xacro" />
     <link name="base_link"/>
     <joint name="base_joint" type="fixed">
@@ -54,9 +54,9 @@
         <parent link="body_link" />
         <child link="lidar_link" />
-        <origin xyz="0.2 0.0 0.0" rpy="0.0 0.0 0.0" />
+        <origin xyz="0.0 0.0 0.1" rpy="0.0 0.0 0.0" />
     </joint>
 	<link name="lidar_link">
 			<visual>
-	  			<origin	xyz="0.0 0.0 0.0" rpy="0.0 0.0 0.0" />
+	  			<origin	xyz="0.0 0.0 0.0" rpy="0.0 0.0 ${PI}" />
       			<geometry>
         			<mesh filename="package://hexapod_description/meshes/phantomX/xv-11_lidar.stl" scale="0.001 0.001 0.001"/>
@@ -88,5 +88,5 @@
     </gazebo>
  	<!-- Attach the pan and tilt head -->
-   	<head name="head_base" parent="body_link" color="White">
+   	<head name="head_base" parent="body" color="White">
       		<origin xyz="${head_offset_x} ${head_offset_y} ${head_offset_z}" rpy="0 0 ${PI}" />
    	</head>
