Commit message: Update xtion.urdf.xacro

File: hexapod_description/urdf/xtion.urdf.xacro (robot description, xacro)
@@ -18,5 +18,5 @@
             <origin xyz="0 0 -0.02" rpy="0 0 0"/>
             <geometry>
-               <mesh filename="package://rbx2_description/meshes/xtion.stl" scale="${camera_mesh_scale} ${camera_mesh_scale} ${camera_mesh_scale}" />
+               <mesh filename="package://hexapod_description/meshes/phantomX/xtion.stl" scale="${camera_mesh_scale} ${camera_mesh_scale} ${camera_mesh_scale}" />
             </geometry>
             <material name="${color}" />

Commit message: modified:   dynamixel_sdk/src/dxl_hal.cpp 	modified:   hexapod_bringup/launch/components/robot_localization_ekf.launch 	modified:   hexapod_bringup/launch/components/rtabmap.launch 	new file:   hexapod_bringup/launch/components/rtabmap_AAC.launch 	modified:   hexapod_bringup/launch/components/rtabmap_AC.launch 	new file:   hexapod_bringup/launch/freenect_throttle.launch 	modified:   hexapod_bringup/launch/hexapod_full.launch 	modified:   hexapod_description/params/joystick_xb.yaml 	modified:   hexapod_description/urdf/pan_tilt_head_xtion.urdf.xacro 	modified:   hexapod_description/urdf/xtion.urdf.xacro

File: hexapod_description/urdf/xtion.urdf.xacro (robot description, xacro)
@@ -29,10 +29,10 @@
          </collision>
       </link>
-      <joint name="camera_depth_joint" type="fixed">
+      <joint name="camera_depth_frame" type="fixed">
           <origin xyz="0 0.025 0" rpy="0 0 0" />
           <parent link="camera_link" />
-          <child link="camera_depth_frame" />
+          <child link="camera_depth_frame_link" />
       </joint>
-      <link name="camera_depth_frame">
+      <link name="camera_depth_frame_link">
       <inertial>
          <mass value="0.000001" />
@@ -43,7 +43,7 @@
          </inertial>
       </link>
-      <joint name="camera_depth_optical_joint" type="fixed">
+      <joint name="camera_depth_joint" type="fixed">
          <origin xyz="0 0 0" rpy="${-PI/2} 0 ${-PI/2}" />
-         <parent link="camera_depth_frame" />
+         <parent link="camera_depth_frame_link" />
          <child link="camera_depth_optical_frame" />
       </joint>
